File: UGR/New_Screen_26/UGR_Driver_Screen_26_PCB/UGR_Driver_Screen_26.kicad_sch (KiCad schematic)
At the start: 59 parts, among them J2 USB_B_Micro, J3 Conn_02x20_Socket, J4 Conn_01x06, U1 TPS562200, U2 STM32F767VGTx, U3 SI2347DS-T1-GE3, U4 MCP2562-E-MF, U5 SI2347DS-T1-GE3, U6 SI2347DS-T1-GE3, U7 SI2347DS-T1-GE3, U8 SI2347DS-T1-GE3, U9 SI2347DS-T1-GE3

Commit message: Rover + UGR Screen PCB
Parts:
- removed D4: BZX384xxxx, Diode_SMD:D_SOD-323, symbol Diode:BZX384xxxx
- removed F1: 0.75A, Fuse:Fuse_1812_4532Metric_Pad1.30x3.40mm_HandSolder, symbol Device:Polyfuse_Small
- removed J2: USB_B_Micro, Connector_USB:USB_Micro-B_Wuerth_629105150521, symbol Connector:USB_B_Micro
- removed J4: Conn_01x06, Connector_PinHeader_2.54mm:PinHeader_1x06_P2.54mm_Vertical, symbol Connector_Generic:Conn_01x06
- removed Main_Conn1: Conn_01x04, UGR:Bulgin_4_Pin, symbol Connector_Generic:Conn_01x04
- removed Main_Conn_Parallel1: Conn_01x04, Connector_PinHeader_2.54mm:PinHeader_1x04_P2.54mm_Vertical, symbol Connector_Generic:Conn_01x04
- removed R1_POWER1, R1_POWER2, R1_POWER3, R1_POWER4, R1_POWER5, R1_POWER6: 47k, Resistor_SMD:R_0603_1608Metric_Pad0.98x0.95mm_HandSolder, symbol Device:R
- removed R1_USB1, R2_USB1: 22R, Resistor_SMD:R_0603_1608Metric_Pad0.98x0.95mm_HandSolder, symbol Device:R
- removed U3, U5, U6, U7, U8, U9: SI2347DS-T1-GE3, SOT_7DS-T1-GE3_VIS, symbol SI2347DS-T1-GE3:SI2347DS-T1-GE3
- removed U4: MCP2562-E-MF, Package_SO:SOIC-8_3.9x4.9mm_P1.27mm, symbol Interface_CAN_LIN:MCP2562-E-MF
- added CONN1: PXP4013/08P/PC, Apps:Bulgin_4000_PXP4013-08S-PC, symbol APPS_Local_Symbols:Bulgin_PXP4013/08P/PC
- added C_SD1, C_TPS1, C_TPS2, C_TPS3: 0.1u, Capacitor_SMD:C_0603_1608Metric_Pad1.08x0.95mm_HandSolder, symbol Device:C_Small
- added D5: BZX384x, Diode_SMD:D_SOD-323, symbol Diode:BZX384xxxx
- added D7: BZX384xxxx, Diode_SMD:D_SOD-323, symbol Diode:BZX384xxxx
- added F2, F3: 0.75A, Fuse:Fuse_1812_4532Metric_Pad1.30x3.40mm_HandSolder, symbol Device:Polyfuse_Small
- added J1: 2171790001, UGR:MOLEX_2171790001, symbol 2171790001:2171790001
- added J2: Conn_01x05, Connector_PinHeader_2.54mm:PinHeader_1x05_P2.54mm_Vertical, symbol Connector_Generic:Conn_01x05
- added J5: Conn_01x06, Connector_PinHeader_2.54mm:PinHeader_1x06_P2.54mm_Vertical, symbol Connector_Generic:Conn_01x06
- added R1_CC1, R2_CC1: 5.1k, Resistor_SMD:R_0603_1608Metric_Pad0.98x0.95mm_HandSolder, symbol Device:R
- added R1_VBUS1: 20k, Resistor_SMD:R_0603_1608Metric_Pad0.98x0.95mm_HandSolder, symbol Device:R
- added R2_VBUS1: 10k, Resistor_SMD:R_0603_1608Metric_Pad0.98x0.95mm_HandSolder, symbol Device:R
- added R_DISCH1: 100k, Resistor_SMD:R_0603_1608Metric_Pad0.98x0.95mm_HandSolder, symbol Device:R
- added R_LIM1: 250, Resistor_SMD:R_0603_1608Metric_Pad0.98x0.95mm_HandSolder, symbol Device:R
- added R_SD1, R_SD2, R_SD5, R_SD6: 10k, Resistor_SMD:R_0603_1608Metric_Pad0.98x0.95mm_HandSolder, symbol Device:R_Small
- added R_SD3, R_SD4: 30k, Resistor_SMD:R_0603_1608Metric_Pad0.98x0.95mm_HandSolder, symbol Device:R_Small
- added TPS2112APW1: ~, UGR:SOP65P640X120-8N, symbol My_ICs:TPS2112APW
- added U3: LM358DT, LM358:SOIC127P600X175-8N, symbol LM358:LM358DT
- added U5: MCP2562-E-SN, Package_SO:SOIC-8_3.9x4.9mm_P1.27mm, symbol Interface_CAN_LIN:MCP2562-E-SN
Connections:
- net 3V3 REG is gone; now on net +3V3: C16_U1.1, C18_U1.1, L2_U1.2, R10_U1.1
- net +3V3: now also U5.5 (Vio)
- net +5V: now also C_SD1.2, C_TPS2.1, J2.1 (Pin_1), TPS2112APW1.7 (OUT), U3.8 (VCC+), U5.3 (VDD)
- net 5V MAIN CON: now also C_TPS1.1, D7.1 (K), F3.2, J5.6 (Pin_6), TPS2112APW1.8 (IN1)
- net 5V USB: now also C_TPS3.1, D5.1 (K), F2.1, R2_VBUS1.1, R_DISCH1.2, TPS2112APW1.6 (IN2)
- net CAN1_RX: now also U5.4 (RXD)
- net CAN1_TX: now also U5.1 (TXD)
- net GND: now also CONN1.8 (Pin_8), C_SD1.1, C_TPS1.2, C_TPS2.2, C_TPS3.2, D5.2 (A), D7.2 (A), J1.A1B12 (GND1), J1.B1A12 (GND2), J2.5 (Pin_5), J5.5 (Pin_5), R1_CC1.1, R1_VBUS1.1, R2_CC1.1, R_DISCH1.1, R_LIM1.2, R_SD1.1, R_SD2.1, R_SD5.2, R_SD6.2, TPS2112APW1.2 (EN_BAR), TPS2112APW1.3 (VSNS), TPS2112APW1.5 (GND), U3.4 (VCC-), U5.2 (VSS), U5.8 (STBY)
- net NRST: now also J2.4 (Pin_4)
- net SWCLK: now also J2.2 (Pin_2)
- net SWDIO: now also J2.3 (Pin_3)
- net T_INT: now also J3.39 (Pin_39)
- net at U2.68 (PA9): now also R1_VBUS1.2, R2_VBUS1.2
- net USB_DN: now reaches U2.70 (PA11)
- net USB_DN: now also J1.A7 (DN1), J1.B7 (DN2)
- net USB_DP: now reaches U2.71 (PA12)
- net USB_DP: now also J1.A6 (DP1), J1.B6 (DP2)
- net CANH renamed CAN_P
- net CAN_P: now also CONN1.5 (Pin_5), J5.4 (Pin_4), U5.7 (CANH)
- net CANL renamed CAN_N
- net CAN_N: now also CONN1.4 (Pin_4), J5.3 (Pin_3), U5.6 (CANL)
- new net: CONN1.3 (Pin_3), F3.1
- new net: R_SD2.2, R_SD4.2, U3.5 (IN2+)
- new net: R_LIM1.1, TPS2112APW1.4 (ILIM)
- new net: R_SD1.2, R_SD3.1, U3.3 (IN1+)
- new net: F2.2, J1.A4B9 (VBUS1), J1.B4A9 (VBUS2)
- new net: J1.A5 (CC1), R1_CC1.2
- new net: J1.B5 (CC2), R2_CC1.2
- new net MCU_SDC+: R_SD6.1, U3.1 (OUT1), U3.2 (IN1-)
- new net MCU_SDC-: R_SD5.1, U3.6 (IN2-), U3.7 (OUT2)
- new net SDC+: CONN1.2 (Pin_2), J5.2 (Pin_2), R_SD3.2
- new net SDC-: CONN1.1 (Pin_1), J5.1 (Pin_1), R_SD4.1
- no-connect marks 55 -> 63
Other:
- note added: "Create common 5V line from USB and MAIN_CONN"
- note added: "DEBUG CON"
- note added: "POWER RAIL OR"
- note added: "SDC READING"
- note removed: "Create common 5V and 3V3 lines from either CAR power or USB power"
- note removed: "POWER RAILS"
- moved on the sheet: ABM3-8.000MHZ-10-1-U-T1, C1_CAP1, C1_OSC1, C1_VDD1, C2_CAP1, C2_OSC1, C2_VDD1, C3_VDD1, C4_VDD1, C5_VDD1, C6_VD1, C8_VDDA1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

Commit message: Screen V2
Parts:
- added J4: DF51-4DP-2DS_50_, DF51:HIROSE_DF51-4DP-2DS_50_, symbol DF51:DF51-4DP-2DS_50_
- added U4, U6: ~, MMBT5551LT1G:SOT95P237X111-3N, symbol MMBT5550L:MMBT5550L
Connections:
- net GND: now also U4.2 (E), U6.2 (E)
- net MCU_SDC+: now also U2.22 (PA0)
- net MCU_SDC-: now also U2.23 (PA1)
- net STATE_RD: now reaches U2.25 (PA3)
- net STATE_RD: now also J4.1
- net DASH_LED_1: now reaches U2.90 (PB4)
- net DASH_LED_1: now also U4.1 (B)
- net DASH_LED_2: now reaches U2.92 (PB6)
- net DASH_LED_2: now also U6.1 (B)
- new net: J4.3, U6.3 (C)
- new net: J4.2, U4.3 (C)
- no-connect marks 63 -> 58
Other:
- note added: "DASHBOARD DF51 INTERFACE"
- moved on the sheet: R1_I2C1, R2_I2C1

Commit message: Screen V2 Rev2
Connections:
- net at R_SD1.2, R_SD3.1: no longer U3.3 (IN1+)
Other:
- moved on the sheet: C10_U1, C12_U1, C14_U1, C16_U1, C18_U1, D2, D3, J4, L2_U1, R10_U1, R11_U1, R5_U1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
