File: UGR/New_Screen_26/UGR_Driver_Screen_26_PCB/_autosave-UGR_Driver_Screen_26.kicad_pcb (KiCad board)
At the start: 2 copper layers, 133.5 x 84 mm, 74 parts, among them J1 2171790001, J2 Conn_01x05, J3 Conn_02x20_Socket, J4 DF51-4DP-2DS_50_, J5 Conn_01x06, U1 TPS562200, U2 STM32F767VGTx, U3 LM358DT, U5 MCP2562-E-SN

Commit message: Screen V2
Parts:
- moved G*** 1.35 mm to (89.5, 91.2)
Connections:
- U2 pad 22: STATE_RD -> MCU_SDC+
- U2 pad 23: unconnected-(U2-PA1-Pad23) -> MCU_SDC-
- U2 pad 24: MCU_SDC+ -> unconnected-(U2-PA2-Pad24)
- U2 pad 25: MCU_SDC- -> STATE_RD
Routing:
- net GND: track 99.5 -> 110.2 mm, vias 101 -> 100
- net T_RST: track 48.4 -> 49.9 mm
- net MCU_SDC-: track 86.8 -> 87.5 mm
- net SWCLK: track 61.6 -> 62.2 mm
- net LCD_RS: track 55.5 -> 55.0 mm

Commit message: Screen V2 Rev2
Parts:
- moved R_LED1 3.76 mm to (83.0, 130.1)
- moved ABM3-8.000MHZ-10-1-U-T1 3.76 mm to (172.0, 126.7)
- moved C10_U1 3.76 mm to (117.5, 117.8)
- moved C14_U1 3.76 mm to (113.0, 112.8)
- moved C16_U1 3.76 mm to (107.5, 107.8)
- moved C18_U1 3.76 mm to (112.0, 107.8)
- moved C1_CAP1 3.76 mm to (182.5, 103.2)
- moved C1_VDD1 3.76 mm to (183.0, 113.7)
- moved C2_CAP1 3.76 mm to (166.2, 97.2)
- moved C2_OSC1 3.76 mm to (175.5, 126.7)
- moved C2_VDD1 3.76 mm to (182.5, 101.2)
- moved C5_VDD1 3.76 mm to (171.0, 119.2)
- moved C6_VD1 3.76 mm to (162.0, 113.7)
- moved C8_VDDA1 3.76 mm to (179.1, 119.2)
- moved C_TPS1 3.76 mm to (93.9, 115.7)
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