File: UGR/New_Screen_26/UGR_Driver_Screen_26_PCB_V2/UGR_Driver_Screen_26.kicad_pcb (KiCad board)
At the start: 2 copper layers, 133.5 x 84 mm, 76 parts, among them J1 2171790001, J2 Conn_01x05, J3 Conn_02x20_Socket, J4 DF51-4DP-2DS_50_, J5 Conn_01x06, U1 TPS562200, U2 STM32F767VGTx, U3 LM358DT, U5 MCP2562-E-SN

Commit message: Screen V2 REV2 changes
Parts:
- moved R1_NRST1 2.53 mm to (130.0, 136.3)
- moved R_DISCH1 1.40 mm to (179.7, 66.3)
- moved R1_CC1 0.91 mm to (169.7, 66.2)
- moved F2 0.80 mm to (173.8, 66.3)
- moved C2_CAP1 0.37 mm to (166.0, 96.9)
- moved USB_C 0.26 mm to (167.6, 59.6)
- moved C3_VDD1 0.24 mm to (164.0, 96.9)
- moved J4 0.15 mm to (116.0, 63.1)
- moved R2_CC1 0.10 mm to (165.7, 66.2)
- moved D5 0.10 mm to (173.4, 71.0)
- renumbered J1 to USB_C
Routing:
- net USB_DP: track 43.7 -> 39.9 mm, vias 2 -> 0
- net USB_DN: track 43.4 -> 39.7 mm, vias 2 -> 0
- net GND: track 139.0 -> 142.6 mm, vias 139 -> 151
- net T_SDA: track 83.3 -> 80.5 mm, vias 4 -> 2
- net T_SCL: track 78.5 -> 76.0 mm, vias 3 -> 1
- net +5V: track 184.9 -> 186.8 mm
- net Net-(U6-C): track 3.45 -> 5.17 mm
- net Net-(J1-VBUS1): track 15.7 -> 17.3 mm
- net +3V3: track 498.6 -> 497.1 mm
- net SWDIO: track 75.1 -> 76.6 mm
- net NRST: track 75.4 -> 74.5 mm, vias 0 -> 2
- net CAN1_RX: track 37.7 -> 38.6 mm, vias 0 -> 2
- net Net-(U2-VCAP_2): track 2.22 -> 3.01 mm
- net Net-(U2-PA9): track 18.3 -> 18.8 mm
- net 5V USB: track 134.0 -> 133.9 mm, vias 6 -> 7
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Other:
- outline, holes or cut-outs redrawn
